File: Supply.sch (KiCad schematic (older format))
At the start: 27 parts, among them IC1 LM5017, IC2 AP65111, U6 7805_SO8

Commit message: - updated project to 5.0.0 - added some more ignores
Parts:
- C10, C11, C12, C27, C30, C31, C32, C45, C48: symbol C -> Device:C
- C28, C46: symbol C_Small -> Device:C_Small
- C49: symbol CP -> Device:CP
- D8: symbol D_Small -> Device:D_Small
- IC1: symbol LM5017 -> Revolter-rescue:LM5017
- IC2: symbol AP65111 -> Revolter-rescue:AP65111
- L1: symbol INDUCTOR -> Revolter-rescue:INDUCTOR
- L2: symbol INDUCTOR_SMALL -> Revolter-rescue:INDUCTOR_SMALL
- R30, R31, R39, R40, R41, R42, R43, R44, R49: symbol R -> Device:R
- U6: symbol 7805_SO8 -> Revolter-rescue:7805_SO8
Changed lines of the file:
@@
-EESchema Schematic File Version 2
-LIBS:Revolter-rescue
-LIBS:power
-LIBS:device
-LIBS:transistors
-LIBS:conn
-LIBS:linear
-LIBS:regul
-LIBS:74xx
-LIBS:cmos4000
-LIBS:adc-dac
-LIBS:memory
-LIBS:xilinx
-LIBS:microcontrollers
-LIBS:dsp
-LIBS:microchip
-LIBS:analog_switches
-LIBS:motorola
-LIBS:texas
-LIBS:intel
-LIBS:audio
-LIBS:interface
-LIBS:digital-audio
-LIBS:philips
-LIBS:display
-LIBS:cypress
-LIBS:siliconi
-LIBS:opto
-LIBS:atmel
-LIBS:contrib
-LIBS:valves
-LIBS:alexlib
+EESchema Schematic File Version 4
 LIBS:Revolter-cache
-EELAYER 25 0
+EELAYER 26 0
 EELAYER END
 $Descr A4 11693 8268
@@
 $EndDescr
 $Comp
-L +12V #PWR052
+L power:+12V #PWR052
 U 1 1 5757C6C9
 P 7500 1650
@@
 $EndComp
 $Comp
-L C C30
+L Device:C C30
 U 1 1 589B52B3
 P 3900 1600
@@
 $EndComp
 $Comp
-L C C31
+L Device:C C31
 U 1 1 589B5758
 P 5850 2050
@@
 $EndComp
 $Comp
-L R R43
+L Device:R R43
 U 1 1 589B6AE0
 P 7500 2200
@@
 $EndComp
 $Comp
-L R R44
+L Device:R R44
 U 1 1 589B6BD8
 P 7500 1900
@@
 $EndComp
 $Comp
-L C C48
+L Device:C C48
 U 1 1 589B6CE4
 P 7200 2050
@@
 $EndComp
 $Comp
-L GND #PWR053
+L power:GND #PWR053
 U 1 1 589B6D8B
 P 5850 2200
@@
 $EndComp
 $Comp
-L INDUCTOR L1
+L Revolter-rescue:INDUCTOR L1
 U 1 1 589B8AC8
 P 6400 1750
@@
 $EndComp
 $Comp
-L C C32
+L Device:C C32
 U 1 1 589B8B47
 P 5850 1600
@@
 $EndComp
 $Comp
-L +5V #PWR054
+L power:+5V #PWR054
 U 1 1 589BAA8C
 P 5550 5050
@@
 $EndComp
 $Comp
-L CP C49
+L Device:CP C49
 U 1 1 589C2A67
 P 6950 2050
@@
 $EndComp
 $Comp
-L LM5017 IC1
+L Revolter-rescue:LM5017 IC1
 U 1 1 59A1C402
 P 5050 1750
@@
 Connection ~ 6950 1750
 $Comp
-L GND #PWR055
+L power:GND #PWR055
 U 1 1 59A1EBF8
 P 6950 2200
@@
 $EndComp
 $Comp
-L GND #PWR056
+L power:GND #PWR056
 U 1 1 59A1EC3C
 P 7200 2200
@@
 $EndComp
 $Comp
-L GND #PWR057
+L power:GND #PWR057
 U 1 1 59A1F45A
 P 7500 2350
@@
 Connection ~ 3900 1450
 $Comp
-L GND #PWR058
+L power:GND #PWR058
 U 1 1 59A204D9
 P 3900 1750
@@
 $EndComp
 $Comp
-L GND #PWR059
+L power:GND #PWR059
 U 1 1 59A20BA8
 P 5150 2400
@@
 $EndComp
 $Comp
-L R R39
+L Device:R R39
 U 1 1 59A20EE3
 P 4450 1600
@@
 Connection ~ 4450 1450
 $Comp
-L GND #PWR060
+L power:GND #PWR060
 U 1 1 59A21253
 P 4950 2400
@@
 $EndComp
 $Comp
-L R R30
+L Device:R R30
 U 1 1 59A216ED
 P 4250 1600
@@
 $EndComp
 $Comp
-L R R31
+L Device:R R31
 U 1 1 59A21733
 P 4250 2050
@@
 	4250 1900 4450 1900
 $Comp
-L GND #PWR061
+L power:GND #PWR061
 U 1 1 59A21882
 P 4250 2200
@@
 Connection ~ 4250 1450
 $Comp
-L D_Small D8
+L Device:D_Small D8
 U 1 1 59A220CE
 P 6350 1450
@@
 Connection ~ 5850 1900
 $Comp
-L R R41
+L Device:R R41
 U 1 1 59A22806
 P 6200 1850
@@
 Connection ~ 6700 1750
 $Comp
-L C_Small C46
+L Device:C_Small C46
 U 1 1 59A22F86
 P 6550 1850
@@
 Connection ~ 6050 1750
 $Comp
-L C_Small C28
+L Device:C_Small C28
 U 1 1 59A2303D
 P 6400 1950
@@
 	6000 1900 5650 1900
 $Comp
-L +12V #PWR062
+L power:+12V #PWR062
 U 1 1 59A25AAF
 P 4300 3500
@@
 $EndComp
 $Comp
-L C C10
+L Device:C C10
 U 1 1 59A25E50
 P 4300 3750
@@
 Connection ~ 4300 3600
 $Comp
-L GND #PWR063
+L power:GND #PWR063
 U 1 1 59A26187
 P 4300 3900
@@
 Connection ~ 4600 3600
 $Comp
-L C C12
+L Device:C C12
 U 1 1 59A2634B
 P 5500 3450
@@
 $EndComp
 $Comp
-L INDUCTOR_SMALL L2
+L Revolter-rescue:INDUCTOR_SMALL L2
 U 1 1 59A263AF
 P 5950 3600
@@
 	5700 3600 5500 3600
 $Comp
-L R R42
+L Device:R R42
 U 1 1 59A2642F
 P 6200 3750
@@
 $EndComp
 $Comp
-L R R49
+L Device:R R49
 U 1 1 59A265EC
 P 6200 4050
@@
 $EndComp
 $Comp
-L GND #PWR064
+L power:GND #PWR064
 U 1 1 59A26636
 P 5050 4200
@@
 $EndComp
 $Comp
-L GND #PWR065
+L power:GND #PWR065
 U 1 1 59A2668D
 P 6200 4200
@@
 	6200 3600 6500 3600
 $Comp
-L C C45
+L Device:C C45
 U 1 1 59A2675E
 P 6500 4050
@@
 $EndComp
 $Comp
-L GND #PWR066
+L power:GND #PWR066
 U 1 1 59A26802
 P 6500 4200
@@
 Connection ~ 6200 3600
 $Comp
-L R R40
+L Device:R R40
 U 1 1 59A26AC7
 P 5950 3900
@@
 Connection ~ 5500 3600
 $Comp
-L +3V3 #PWR067
+L power:+3V3 #PWR067
 U 1 1 59A27760
 P 6500 3500
@@
 Connection ~ 6500 3600
 $Comp
-L +12V #PWR068
+L power:+12V #PWR068
 U 1 1 59A27DFE
 P 4600 5050
@@
 $EndComp
 $Comp
-L C C11
+L Device:C C11
 U 1 1 59A27E04
 P 4600 5300
@@
 Connection ~ 4600 5150
 $Comp
-L GND #PWR069
+L power:GND #PWR069
 U 1 1 59A27E0D
 P 4600 5450
@@
 $EndComp
 $Comp
-L C C27
+L Device:C C27
 U 1 1 59A28622
 P 5550 5300
@@
 Connection ~ 5550 5150
 $Comp
-L GND #PWR070
+L power:GND #PWR070
 U 1 1 59A2862B
 P 5550 5450
@@
 $EndComp
 $Comp
-L GND #PWR071
+L power:GND #PWR071
 U 1 1 59A28C15
 P 5100 5450
@@
 $EndComp
 $Comp
-L 7805_SO8 U6
+L Revolter-rescue:7805_SO8 U6
 U 1 1 59BF7E66
 P 5050 5200
+AR Path="/59BF7E66" Ref="U6"  Part="1"
+AR Path="/5899E25F/59BF7E66" Ref="U6"  Part="1"
 F 0 "U6" H 5200 5004 50  0000 C CNN
 F 1 "7805_SO8" H 5050 5400 50  0000 C CNN
@@
 $EndComp
 $Comp
-L GND #PWR072
+L power:GND #PWR072
 U 1 1 59BF9EB5
 P 4950 5450
@@
 $EndComp
 $Comp
-L GND #PWR073
+L power:GND #PWR073
 U 1 1 59BF9F14
 P 5000 5450
@@
 $EndComp
 $Comp
-L GND #PWR074
+L power:GND #PWR074
 U 1 1 59BFA02F
 P 5150 5450
@@
 $EndComp
 $Comp
-L +BATT #PWR075
+L power:+BATT #PWR075
 U 1 1 59C14A31
 P 3900 1300
@@
 	3900 1300 3900 1450
 $Comp
-L AP65111 IC2
+L Revolter-rescue:AP65111 IC2
 U 1 1 5A89C59A
 P 5050 3600

Commit message: - swapped TO220 dual MOSFET for single DualCool88 MOSFET package - removed postdriver - changed IRS2110 for IRS2186 - added third shunt - rewired CPU for VESC6 compatibility - layout completely from scratch
Parts:
- C10, C11, C12, C27, C28, C31, C32, C45, C46, C48: footprint Capacitors_SMD:C_0805 -> Capacitor_SMD:C_0805_2012Metric
- C30: footprint Capacitors_SMD:C_1206 -> Capacitor_SMD:C_1206_3216Metric
- C49: footprint Capacitors_THT:CP_Radial_D6.3mm_P2.50mm -> Capacitor_THT:CP_Radial_D6.3mm_P2.50mm
- D8: footprint Diodes_SMD:D_MiniMELF_Standard -> Diode_SMD:D_MiniMELF
- IC1: footprint Housings_SOIC:SOIC-8-1EP_3.9x4.9mm_Pitch1.27mm -> Package_SO:HSOP-8-1EP_3.9x4.9mm_P1.27mm_EP2.41x3.1mm
- IC2: footprint TO_SOT_Packages_SMD:SOT-23-6 -> Package_TO_SOT_SMD:SOT-23-6
- L1: footprint alexmod:VLS6045EX -> Inductor_SMD:L_Taiyo-Yuden_NR-60xx_HandSoldering
- L2: footprint alexmod:NRH2410 -> Inductor_SMD:L_Taiyo-Yuden_NR-24xx_HandSoldering
- R30, R31, R39, R40, R41, R42, R43, R44, R49: footprint Resistors_SMD:R_0805 -> Resistor_SMD:R_0805_2012Metric
- U6: footprint Housings_SOIC:SOIC-8_3.9x4.9mm_Pitch1.27mm -> Package_SO:SO-8_3.9x4.9mm_P1.27mm
Changed lines of the file:
@@
 $Descr A4 11693 8268
 encoding utf-8
-Sheet 6 7
+Sheet 5 7
 Title ""
 Date ""
@@
 F 0 "C30" H 3925 1700 50  0000 L CNN
 F 1 "1u" H 3925 1500 50  0000 L CNN
-F 2 "Capacitors_SMD:C_1206" H 3938 1450 50  0001 C CNN
+F 2 "Capacitor_SMD:C_1206_3216Metric" H 3938 1450 50  0001 C CNN
 F 3 "" H 3900 1600 50  0000 C CNN
 	1    3900 1600
@@
 F 0 "C31" H 5875 2150 50  0000 L CNN
 F 1 "100n" H 5875 1950 50  0000 L CNN
-F 2 "Capacitors_SMD:C_0805" H 5888 1900 50  0001 C CNN
+F 2 "Capacitor_SMD:C_0805_2012Metric" H 5888 1900 50  0001 C CNN
 F 3 "" H 5850 2050 50  0000 C CNN
 	1    5850 2050
@@
 F 0 "R43" V 7580 2200 50  0000 C CNN
 F 1 "1k" V 7500 2200 50  0000 C CNN
-F 2 "Resistors_SMD:R_0805" V 7430 2200 50  0001 C CNN
+F 2 "Resistor_SMD:R_0805_2012Metric" V 7430 2200 50  0001 C CNN
 F 3 "" H 7500 2200 50  0000 C CNN
 	1    7500 2200
@@
 F 0 "R44" V 7580 1900 50  0000 C CNN
 F 1 "10k" V 7500 1900 50  0000 C CNN
-F 2 "Resistors_SMD:R_0805" V 7430 1900 50  0001 C CNN
+F 2 "Resistor_SMD:R_0805_2012Metric" V 7430 1900 50  0001 C CNN
 F 3 "" H 7500 1900 50  0000 C CNN
 	1    7500 1900
@@
 F 0 "C48" H 7225 2150 50  0000 L CNN
 F 1 "22u" H 7225 1950 50  0000 L CNN
-F 2 "Capacitors_SMD:C_0805" H 7238 1900 50  0001 C CNN
+F 2 "Capacitor_SMD:C_0805_2012Metric" H 7238 1900 50  0001 C CNN
 F 3 "" H 7200 2050 50  0000 C CNN
 	1    7200 2050
@@
 F 0 "L1" V 6350 1750 50  0000 C CNN
 F 1 "VLS6045EX-221M" V 6500 1750 50  0000 C CNN
-F 2 "alexmod:VLS6045EX" H 6400 1750 50  0001 C CNN
+F 2 "Inductor_SMD:L_Taiyo-Yuden_NR-60xx_HandSoldering" H 6400 1750 50  0001 C CNN
 F 3 "" H 6400 1750 50  0000 C CNN
 	1    6400 1750
@@
 F 0 "C32" H 5875 1700 50  0000 L CNN
 F 1 "100n" H 5875 1500 50  0000 L CNN
-F 2 "Capacitors_SMD:C_0805" H 5888 1450 50  0001 C CNN
+F 2 "Capacitor_SMD:C_0805_2012Metric" H 5888 1450 50  0001 C CNN
 F 3 "" H 5850 1600 50  0000 C CNN
 	1    5850 1600
@@
 F 0 "C49" H 6975 2150 50  0000 L CNN
 F 1 "100u 22V" H 6975 1950 50  0000 L CNN
-F 2 "Capacitors_THT:CP_Radial_D6.3mm_P2.50mm" H 6988 1900 50  0001 C CNN
+F 2 "Capacitor_THT:CP_Radial_D6.3mm_P2.50mm" H 6988 1900 50  0001 C CNN
 F 3 "" H 6950 2050 50  0000 C CNN
 	1    6950 2050
@@
 F 0 "IC1" H 5050 1750 60  0000 C CNN
 F 1 "LM5017" H 5050 1900 60  0000 C CNN
-F 2 "Housings_SOIC:SOIC-8-1EP_3.9x4.9mm_Pitch1.27mm" H 5050 1600 60  0001 C CNN
+F 2 "Package_SO:HSOP-8-1EP_3.9x4.9mm_P1.27mm_EP2.41x3.1mm" H 5050 1600 60  0001 C CNN
 F 3 "" H 5050 1600 60  0000 C CNN
 	1    5050 1750
@@
 $EndComp
 Wire Wire Line
-	5650 1750 6100 1750
+	5650 1750 5850 1750
 Connection ~ 5850 1750
 Wire Wire Line
@@
 	7200 1750 7200 1900
 Wire Wire Line
-	6700 1750 7500 1750
+	6700 1750 6950 1750
 Connection ~ 6950 1750
 $Comp
@@
 Connection ~ 7500 1750
 Wire Wire Line
-	3900 1450 4450 1450
+	3900 1450 4250 1450
 Connection ~ 3900 1450
 $Comp
@@
 F 0 "R39" V 4530 1600 50  0000 C CNN
 F 1 "499k" V 4450 1600 50  0000 C CNN
-F 2 "Resistors_SMD:R_0805" V 4380 1600 50  0001 C CNN
+F 2 "Resistor_SMD:R_0805_2012Metric" V 4380 1600 50  0001 C CNN
 F 3 "" H 4450 1600 50  0000 C CNN
 	1    4450 1600
@@
 F 0 "R30" V 4330 1600 50  0000 C CNN
 F 1 "82k" V 4250 1600 50  0000 C CNN
-F 2 "Resistors_SMD:R_0805" V 4180 1600 50  0001 C CNN
+F 2 "Resistor_SMD:R_0805_2012Metric" V 4180 1600 50  0001 C CNN
 F 3 "" H 4250 1600 50  0000 C CNN
 	1    4250 1600
@@
 F 0 "R31" V 4330 2050 50  0000 C CNN
 F 1 "10k" V 4250 2050 50  0000 C CNN
-F 2 "Resistors_SMD:R_0805" V 4180 2050 50  0001 C CNN
+F 2 "Resistor_SMD:R_0805_2012Metric" V 4180 2050 50  0001 C CNN
 F 3 "" H 4250 2050 50  0000 C CNN
 	1    4250 2050
@@
 F 0 "D8" H 6300 1530 50  0000 L CNN
 F 1 "4148" H 6300 1350 50  0000 L CNN
-F 2 "Diodes_SMD:D_MiniMELF_Standard" V 6350 1450 50  0001 C CNN
+F 2 "Diode_SMD:D_MiniMELF" V 6350 1450 50  0001 C CNN
 F 3 "" V 6350 1450 50  0000 C CNN
 	1    6350 1450
@@
 F 0 "R41" V 6280 1850 50  0000 C CNN
 F 1 "46k4" V 6200 1850 50  0000 C CNN
-F 2 "Resistors_SMD:R_0805" V 6130 1850 50  0001 C CNN
+F 2 "Resistor_SMD:R_0805_2012Metric" V 6130 1850 50  0001 C CNN
 F 3 "" H 6200 1850 50  0000 C CNN
 	1    6200 1850
@@
 $EndComp
 Wire Wire Line
-	6700 1450 6700 1850
+	6700 1450 6700 1750
 Connection ~ 6700 1750
 $Comp
@@
 F 0 "C46" V 6600 1900 50  0000 L CNN
 F 1 "3n3" V 6700 1850 50  0000 L CNN
-F 2 "Capacitors_SMD:C_0805" H 6550 1850 50  0001 C CNN
+F 2 "Capacitor_SMD:C_0805_2012Metric" H 6550 1850 50  0001 C CNN
 F 3 "" H 6550 1850 50  0000 C CNN
 	1    6550 1850
@@
 F 0 "C28" H 6500 2000 50  0000 L CNN
 F 1 "100n" H 6350 2100 50  0000 L CNN
-F 2 "Capacitors_SMD:C_0805" H 6400 1950 50  0001 C CNN
+F 2 "Capacitor_SMD:C_0805_2012Metric" H 6400 1950 50  0001 C CNN
 F 3 "" H 6400 1950 50  0000 C CNN
 	1    6400 1950
@@
 $EndComp
 Wire Wire Line
-	6350 1850 6450 1850
+	6350 1850 6400 1850
 Connection ~ 6400 1850
 Connection ~ 6400 2050
@@
 	6700 1450 6450 1450
 Wire Wire Line
-	5650 2050 7500 2050
+	5650 2050 6400 2050
 Wire Wire Line
 	6250 1450 6000 1450
@@
 	6000 1450 6000 1900
 Wire Wire Line
-	6000 1900 5650 1900
+	6000 1900 5850 1900
 $Comp
 L power:+12V #PWR062
@@
 F 0 "C10" H 4325 3850 50  0000 L CNN
 F 1 "22u" H 4325 3650 50  0000 L CNN
-F 2 "Capacitors_SMD:C_0805" H 4338 3600 50  0001 C CNN
+F 2 "Capacitor_SMD:C_0805_2012Metric" H 4338 3600 50  0001 C CNN
 F 3 "" H 4300 3750 50  0000 C CNN
 	1    4300 3750
@@
 F 0 "C12" H 5525 3550 50  0000 L CNN
 F 1 "100n" H 5525 3350 50  0000 L CNN
-F 2 "Capacitors_SMD:C_0805" H 5538 3300 50  0001 C CNN
+F 2 "Capacitor_SMD:C_0805_2012Metric" H 5538 3300 50  0001 C CNN
 F 3 "" H 5500 3450 50  0000 C CNN
 	1    5500 3450
@@
 F 0 "L2" H 5950 3700 50  0000 C CNN
 F 1 "NRH2410T100MN" H 6050 3800 50  0000 C CNN
-F 2 "alexmod:NRH2410" H 5950 3600 50  0001 C CNN
+F 2 "Inductor_SMD:L_Taiyo-Yuden_NR-24xx_HandSoldering" H 5950 3600 50  0001 C CNN
 F 3 "" H 5950 3600 50  0000 C CNN
 	1    5950 3600
@@
 F 0 "R42" V 6280 3750 50  0000 C CNN
 F 1 "40k2" V 6200 3750 50  0000 C CNN
-F 2 "Resistors_SMD:R_0805" V 6130 3750 50  0001 C CNN
+F 2 "Resistor_SMD:R_0805_2012Metric" V 6130 3750 50  0001 C CNN
 F 3 "" H 6200 3750 50  0000 C CNN
 	1    6200 3750
@@
 F 0 "R49" V 6280 4050 50  0000 C CNN
 F 1 "13k" V 6200 4050 50  0000 C CNN
-F 2 "Resistors_SMD:R_0805" V 6130 4050 50  0001 C CNN
+F 2 "Resistor_SMD:R_0805_2012Metric" V 6130 4050 50  0001 C CNN
 F 3 "" H 6200 4050 50  0000 C CNN
 	1    6200 4050
@@
 F 0 "C45" H 6525 4150 50  0000 L CNN
 F 1 "22u" H 6525 3950 50  0000 L CNN
-F 2 "Capacitors_SMD:C_0805" H 6538 3900 50  0001 C CNN
+F 2 "Capacitor_SMD:C_0805_2012Metric" H 6538 3900 50  0001 C CNN
 F 3 "" H 6500 4050 50  0000 C CNN
 	1    6500 4050
@@
 $EndComp
 Wire Wire Line
-	6500 3500 6500 3900
+	6500 3500 6500 3600
 Connection ~ 6200 3600
 $Comp
@@
 F 0 "R40" V 6030 3900 50  0000 C CNN
 F 1 "59k" V 5950 3900 50  0000 C CNN
-F 2 "Resistors_SMD:R_0805" V 5880 3900 50  0001 C CNN
+F 2 "Resistor_SMD:R_0805_2012Metric" V 5880 3900 50  0001 C CNN
 F 3 "" H 5950 3900 50  0000 C CNN
 	1    5950 3900
@@
 F 0 "C11" H 4625 5400 50  0000 L CNN
 F 1 "100n" H 4625 5200 50  0000 L CNN
-F 2 "Capacitors_SMD:C_0805" H 4638 5150 50  0001 C CNN
+F 2 "Capacitor_SMD:C_0805_2012Metric" H 4638 5150 50  0001 C CNN
 F 3 "" H 4600 5300 50  0000 C CNN
 	1    4600 5300
@@
 F 0 "C27" H 5575 5400 50  0000 L CNN
 F 1 "100n" H 5575 5200 50  0000 L CNN
-F 2 "Capacitors_SMD:C_0805" H 5588 5150 50  0001 C CNN
+F 2 "Capacitor_SMD:C_0805_2012Metric" H 5588 5150 50  0001 C CNN
 F 3 "" H 5550 5300 50  0000 C CNN
 	1    5550 5300
@@
 F 0 "U6" H 5200 5004 50  0000 C CNN
 F 1 "7805_SO8" H 5050 5400 50  0000 C CNN
-F 2 "Housings_SOIC:SOIC-8_3.9x4.9mm_Pitch1.27mm" H 5050 5200 50  0001 C CNN
+F 2 "Package_SO:SO-8_3.9x4.9mm_P1.27mm" H 5050 5200 50  0001 C CNN
 F 3 "" H 5050 5200 50  0000 C CNN
 	1    5050 5200
@@
 F 0 "IC2" H 5050 3500 60  0000 C CNN
 F 1 "AP65111" H 5050 3750 60  0000 C CNN
-F 2 "TO_SOT_Packages_SMD:SOT-23-6" H 5050 3400 60  0001 C CNN
+F 2 "Package_TO_SOT_SMD:SOT-23-6" H 5050 3400 60  0001 C CNN
 F 3 "" H 5050 3400 60  0000 C CNN
 	1    5050 3600
 	1    0    0    -1
 $EndComp
+Wire Wire Line
+	5850 1750 6050 1750
+Wire Wire Line
+	6950 1750 7200 1750
+Wire Wire Line
+	7200 1750 7500 1750
+Wire Wire Line
+	4250 1450 4450 1450
+Wire Wire Line
+	5850 1900 5650 1900
+Wire Wire Line
+	6700 1750 6700 1850
+Wire Wire Line
+	6050 1750 6100 1750
+Wire Wire Line
+	6400 1850 6450 1850
+Wire Wire Line
+	6400 2050 7500 2050
+Wire Wire Line
+	6500 3600 6500 3900
 $EndSCHEMATC
