File: Supply.sch (KiCad schematic (older format))
At the start: 8 parts, among them IC2 AP65111

Commit message: - fixed EN pin of DCDC being forced to VIN (overvoltage)
Parts:
- added R4: 100k, Resistor_SMD:R_0805_2012Metric, symbol Device:R
Connections:
- wire segments 17 -> 18
Other:
- moved on the sheet: C10
Changed lines of the file:
@@
 L power:+12V #PWR062
 U 1 1 59A25AAF
-P 4300 3500
-F 0 "#PWR062" H 4300 3350 50  0001 C CNN
-F 1 "+12V" H 4300 3640 50  0000 C CNN
-F 2 "" H 4300 3500 60  0000 C CNN
-F 3 "" H 4300 3500 60  0000 C CNN
-	1    4300 3500
+P 4000 3500
+F 0 "#PWR062" H 4000 3350 50  0001 C CNN
+F 1 "+12V" H 4000 3640 50  0000 C CNN
+F 2 "" H 4000 3500 60  0000 C CNN
+F 3 "" H 4000 3500 60  0000 C CNN
+	1    4000 3500
 	1    0    0    -1
 $EndComp
@@
 L Device:C C10
 U 1 1 59A25E50
-P 4300 3750
-F 0 "C10" H 4325 3850 50  0000 L CNN
-F 1 "22u" H 4325 3650 50  0000 L CNN
-F 2 "Capacitor_SMD:C_0805_2012Metric" H 4338 3600 50  0001 C CNN
-F 3 "" H 4300 3750 50  0000 C CNN
-	1    4300 3750
+P 4000 3750
+F 0 "C10" H 4025 3850 50  0000 L CNN
+F 1 "22u" H 4025 3650 50  0000 L CNN
+F 2 "Capacitor_SMD:C_0805_2012Metric" H 4038 3600 50  0001 C CNN
+F 3 "" H 4000 3750 50  0000 C CNN
+	1    4000 3750
 	-1   0    0    -1
 $EndComp
 Wire Wire Line
-	4300 3600 4600 3600
+	4000 3600 4300 3600
 $Comp
 L power:GND #PWR063
 U 1 1 59A26187
-P 4300 3900
-F 0 "#PWR063" H 4300 3650 50  0001 C CNN
-F 1 "GND" H 4300 3750 50  0000 C CNN
-F 2 "" H 4300 3900 60  0000 C CNN
-F 3 "" H 4300 3900 60  0000 C CNN
-	1    4300 3900
+P 4000 3900
+F 0 "#PWR063" H 4000 3650 50  0001 C CNN
+F 1 "GND" H 4000 3750 50  0000 C CNN
+F 2 "" H 4000 3900 60  0000 C CNN
+F 3 "" H 4000 3900 60  0000 C CNN
+	1    4000 3900
 	1    0    0    -1
 $EndComp
@@
 L power:+BATT #PWR075
 U 1 1 59C14A31
-P 4000 3500
-F 0 "#PWR075" H 4000 3350 50  0001 C CNN
-F 1 "+BATT" H 4000 3640 50  0000 C CNN
-F 2 "" H 4000 3500 50  0000 C CNN
-F 3 "" H 4000 3500 50  0000 C CNN
-	1    4000 3500
+P 3700 3500
+F 0 "#PWR075" H 3700 3350 50  0001 C CNN
+F 1 "+BATT" H 3700 3640 50  0000 C CNN
+F 2 "" H 3700 3500 50  0000 C CNN
+F 3 "" H 3700 3500 50  0000 C CNN
+	1    3700 3500
 	1    0    0    -1
 $EndComp
@@
 	6500 3600 6500 3900
 Wire Wire Line
-	4600 3800 4600 3600
-Connection ~ 4600 3600
-Wire Wire Line
 	5400 3600 5450 3600
 Wire Wire Line
@@
 Connection ~ 6200 3600
 Wire Wire Line
-	4300 3500 4300 3600
+	4000 3500 4000 3600
+Connection ~ 4000 3600
+Wire Wire Line
+	4000 3600 3700 3600
+Wire Wire Line
+	3700 3600 3700 3500
+$Comp
+L Device:R R4
+U 1 1 610FCFCE
+P 4450 3800
+F 0 "R4" V 4530 3800 50  0000 C CNN
+F 1 "100k" V 4450 3800 50  0000 C CNN
+F 2 "Resistor_SMD:R_0805_2012Metric" V 4380 3800 50  0001 C CNN
+F 3 "" H 4450 3800 50  0000 C CNN
+	1    4450 3800
+	0    1    1    0
+$EndComp
+Wire Wire Line
+	4300 3800 4300 3600
 Connection ~ 4300 3600
 Wire Wire Line
-	4300 3600 4000 3600
-Wire Wire Line
-	4000 3600 4000 3500
+	4300 3600 4600 3600
 $EndSCHEMATC
