File: CAN.sch (KiCad schematic (older format))
At the start: 7 parts, among them IC1 ADM3052

Commit message: - removed 1 MOSFET of each group (no space) - removed 2 DC buffer caps (no space) - power stage routed - shunts and amps routed - post driver routed - pre driver HV routed
Parts:
- removed C10: 10u, Capacitors_SMD:C_0805, symbol C_Small
- removed C11, C12: 100n, Capacitors_SMD:C_0805, symbol C_Small
- removed C9: 1u, Capacitors_SMD:C_0805, symbol C_Small
- removed IC1: ADM3052, Housings_SOIC:SOIC-16_7.5x10.3mm_Pitch1.27mm, symbol ADM3052
- removed R30: 120R, Resistors_SMD:R_0805, symbol R_Small
- removed R31: 300R, Resistors_SMD:R_1206, symbol R_Small
- added C9: 100n, Capacitors_SMD:C_0805, symbol C
- added U5: PCA82C251, Housings_SOIC:SOIC-8_3.9x4.9mm_Pitch1.27mm, symbol PCA82C251
Connections:
- net labels added: +5V
- net labels removed: +12VA, +3V3, Earth, V+Sense
- wire segments 4 -> 2
Changed lines of the file:
@@
 LIBS:contrib
 LIBS:valves
+LIBS:alexlib
 LIBS:Revolter-cache
 EELAYER 25 0
@@
 Comment4 ""
 $EndDescr
-Text HLabel 6650 3350 2    60   Output ~ 0
+Text HLabel 5350 3200 0    60   Input ~ 0
+CANL
+Text HLabel 5350 3100 0    60   Input ~ 0
+CANH
+Text HLabel 6150 3100 2    60   Input ~ 0
+CAN_TX
+Text HLabel 6150 3500 2    60   Output ~ 0
 CAN_RX
-Text HLabel 6650 3150 2    60   Input ~ 0
-CAN_TX
-Text HLabel 5150 3150 0    60   Input ~ 0
-CANH
-Text HLabel 5150 3350 0    60   Input ~ 0
-CANL
 $Comp
-L ADM3052 IC1
-U 1 1 5759CEA3
-P 6000 3850
-F 0 "IC1" H 6000 3850 60  0000 C CNN
-F 1 "ADM3052" H 6000 4500 60  0000 C CNN
-F 2 "Housings_SOIC:SOIC-16_7.5x10.3mm_Pitch1.27mm" H 6150 3950 60  0001 C CNN
-F 3 "" H 6150 3950 60  0000 C CNN
-	1    6000 3850
+L PCA82C251 U5
+U 1 1 59A31FD5
+P 5750 3200
+F 0 "U5" H 5550 3750 50  0000 L CNN
+F 1 "PCA82C251" H 5550 3650 50  0000 L CNN
+F 2 "Housings_SOIC:SOIC-8_3.9x4.9mm_Pitch1.27mm" H 5750 3150 50  0001 C CNN
+F 3 "" H 5750 3150 50  0000 C CNN
+	1    5750 3200
 	-1   0    0    -1
 $EndComp
 $Comp
-L C_Small C9
-U 1 1 5759CF39
-P 5350 3900
-F 0 "C9" H 5500 4000 50  0000 L CNN
-F 1 "1u" H 5500 3900 50  0000 L CNN
-F 2 "Capacitors_SMD:C_0805" H 5350 3900 60  0001 C CNN
-F 3 "" H 5350 3900 60  0000 C CNN
-	1    5350 3900
-	-1   0    0    -1
-$EndComp
-$Comp
-L C_Small C10
-U 1 1 5759CF9E
-P 5350 4200
-F 0 "C10" H 5450 4250 50  0000 L CNN
-F 1 "10u" H 5450 4150 50  0000 L CNN
-F 2 "Capacitors_SMD:C_0805" H 5350 4200 60  0001 C CNN
-F 3 "" H 5350 4200 60  0000 C CNN
-	1    5350 4200
-	-1   0    0    -1
-$EndComp
-Connection ~ 5350 4100
-Connection ~ 5350 4300
-$Comp
-L R_Small R31
-U 1 1 5759CFE0
-P 5350 4400
-F 0 "R31" V 5250 4350 50  0000 L CNN
-F 1 "300R" H 5400 4400 50  0000 L CNN
-F 2 "Resistors_SMD:R_1206" H 5350 4400 60  0001 C CNN
-F 3 "" H 5350 4400 60  0000 C CNN
-	1    5350 4400
-	-1   0    0    -1
-$EndComp
-$Comp
-L C_Small C11
-U 1 1 5759D08A
-P 5350 4600
-F 0 "C11" H 5500 4600 50  0000 L CNN
-F 1 "100n" H 5450 4500 50  0000 L CNN
-F 2 "Capacitors_SMD:C_0805" H 5350 4600 60  0001 C CNN
-F 3 "" H 5350 4600 60  0000 C CNN
-	1    5350 4600
-	-1   0    0    -1
-$EndComp
-Connection ~ 5350 4500
-$Comp
-L Earth #PWR029
-U 1 1 5759DCFE
-P 5350 4700
-F 0 "#PWR029" H 5350 4450 50  0001 C CNN
-F 1 "Earth" H 5350 4550 50  0001 C CNN
-F 2 "" H 5350 4700 60  0000 C CNN
-F 3 "" H 5350 4700 60  0000 C CNN
-	1    5350 4700
-	-1   0    0    -1
-$EndComp
-$Comp
-L Earth #PWR030
-U 1 1 5759DF52
-P 5350 4100
-F 0 "#PWR030" H 5350 3850 50  0001 C CNN
-F 1 "Earth" H 5350 3950 50  0001 C CNN
-F 2 "" H 5350 4100 60  0000 C CNN
-F 3 "" H 5350 4100 60  0000 C CNN
-	1    5350 4100
-	0    1    -1   0
-$EndComp
-$Comp
-L +12VA #PWR031
-U 1 1 5759E22F
-P 5350 4500
-F 0 "#PWR031" H 5350 4350 50  0001 C CNN
-F 1 "+12VA" V 5350 4750 50  0000 C CNN
-F 2 "" H 5350 4500 60  0000 C CNN
-F 3 "" H 5350 4500 60  0000 C CNN
-	1    5350 4500
-	0    -1   -1   0
-$EndComp
-$Comp
-L GND #PWR032
-U 1 1 5759E8F5
-P 6650 4500
-F 0 "#PWR032" H 6650 4250 50  0001 C CNN
-F 1 "GND" H 6650 4350 50  0000 C CNN
-F 2 "" H 6650 4500 60  0000 C CNN
-F 3 "" H 6650 4500 60  0000 C CNN
-	1    6650 4500
+L +5V #PWR027
+U 1 1 59A3205A
+P 6300 2800
+F 0 "#PWR027" H 6300 2650 50  0001 C CNN
+F 1 "+5V" H 6300 2940 50  0000 C CNN
+F 2 "" H 6300 2800 50  0000 C CNN
+F 3 "" H 6300 2800 50  0000 C CNN
+	1    6300 2800
 	1    0    0    -1
 $EndComp
 $Comp
-L R_Small R30
-U 1 1 5759ED7A
-P 5350 3250
-F 0 "R30" V 5250 3200 50  0000 L CNN
-F 1 "120R" H 5400 3250 50  0000 L CNN
-F 2 "Resistors_SMD:R_0805" H 5350 3250 60  0001 C CNN
-F 3 "" H 5350 3250 60  0000 C CNN
-	1    5350 3250
-	-1   0    0    -1
-$EndComp
-Wire Wire Line
-	5150 3350 5350 3350
-Wire Wire Line
-	5350 3150 5150 3150
-Connection ~ 5350 3150
-Connection ~ 5350 3350
-Text HLabel 6650 3550 2    60   Output ~ 0
-V+Sense
-$Comp
-L C_Small C12
-U 1 1 575A0498
-P 6650 4200
-F 0 "C12" H 6800 4200 50  0000 L CNN
-F 1 "100n" H 6750 4100 50  0000 L CNN
-F 2 "Capacitors_SMD:C_0805" H 6650 4200 60  0001 C CNN
-F 3 "" H 6650 4200 60  0000 C CNN
-	1    6650 4200
+L C C9
+U 1 1 59A32070
+P 6300 3750
+F 0 "C9" H 6325 3850 50  0000 L CNN
+F 1 "100n" H 6325 3650 50  0000 L CNN
+F 2 "Capacitors_SMD:C_0805" H 6338 3600 50  0001 C CNN
+F 3 "" H 6300 3750 50  0000 C CNN
+	1    6300 3750
 	1    0    0    -1
 $EndComp
-Connection ~ 6650 4300
-Connection ~ 6650 4500
 $Comp
-L +3V3 #PWR033
-U 1 1 575A0BC8
-P 6650 4100
-F 0 "#PWR033" H 6650 3950 50  0001 C CNN
-F 1 "+3V3" H 6650 4240 50  0000 C CNN
-F 2 "" H 6650 4100 60  0000 C CNN
-F 3 "" H 6650 4100 60  0000 C CNN
-	1    6650 4100
+L GND #PWR028
+U 1 1 59A320DF
+P 5350 3500
+F 0 "#PWR028" H 5350 3250 50  0001 C CNN
+F 1 "GND" H 5350 3350 50  0000 C CNN
+F 2 "" H 5350 3500 50  0000 C CNN
+F 3 "" H 5350 3500 50  0000 C CNN
+	1    5350 3500
+	1    0    0    -1
+$EndComp
+$Comp
+L GND #PWR029
+U 1 1 59A320F7
+P 6300 3900
+F 0 "#PWR029" H 6300 3650 50  0001 C CNN
+F 1 "GND" H 6300 3750 50  0000 C CNN
+F 2 "" H 6300 3900 50  0000 C CNN
+F 3 "" H 6300 3900 50  0000 C CNN
+	1    6300 3900
 	1    0    0    -1
 $EndComp
 Wire Wire Line
-	6650 4300 6650 4500
-Connection ~ 6650 4400
+	6300 2800 6300 3600
 Wire Wire Line
-	5350 4000 5350 4100
-Connection ~ 5350 4000
-Connection ~ 6650 4100
+	6300 2900 6150 2900
+Connection ~ 6300 2900
 $EndSCHEMATC

Commit message: - updated project to 5.0.0 - added some more ignores
Parts:
- C9: symbol C -> Device:C
- U5: symbol PCA82C251 -> philips:PCA82C251
Changed lines of the file:
@@
-EESchema Schematic File Version 2
-LIBS:Revolter-rescue
-LIBS:power
-LIBS:device
-LIBS:transistors
-LIBS:conn
-LIBS:linear
-LIBS:regul
-LIBS:74xx
-LIBS:cmos4000
-LIBS:adc-dac
-LIBS:memory
-LIBS:xilinx
-LIBS:microcontrollers
-LIBS:dsp
-LIBS:microchip
-LIBS:analog_switches
-LIBS:motorola
-LIBS:texas
-LIBS:intel
-LIBS:audio
-LIBS:interface
-LIBS:digital-audio
-LIBS:philips
-LIBS:display
-LIBS:cypress
-LIBS:siliconi
-LIBS:opto
-LIBS:atmel
-LIBS:contrib
-LIBS:valves
-LIBS:alexlib
+EESchema Schematic File Version 4
 LIBS:Revolter-cache
-EELAYER 25 0
+EELAYER 26 0
 EELAYER END
 $Descr A4 11693 8268
@@
 CAN_RX
 $Comp
-L PCA82C251 U5
+L philips:PCA82C251 U5
 U 1 1 59A31FD5
 P 5750 3200
@@
 $EndComp
 $Comp
-L +5V #PWR031
+L power:+5V #PWR031
 U 1 1 59A3205A
 P 6300 2800
@@
 $EndComp
 $Comp
-L C C9
+L Device:C C9
 U 1 1 59A32070
 P 6300 3750
@@
 $EndComp
 $Comp
-L GND #PWR032
+L power:GND #PWR032
 U 1 1 59A320DF
 P 5350 3500
@@
 $EndComp
 $Comp
-L GND #PWR033
+L power:GND #PWR033
 U 1 1 59A320F7
 P 6300 3900

Commit message: - swapped TO220 dual MOSFET for single DualCool88 MOSFET package - removed postdriver - changed IRS2110 for IRS2186 - added third shunt - rewired CPU for VESC6 compatibility - layout completely from scratch
Parts:
- C9: footprint Capacitors_SMD:C_0805 -> Capacitor_SMD:C_0805_2012Metric
- U5: footprint Housings_SOIC:SOIC-8_3.9x4.9mm_Pitch1.27mm -> Package_SO:SO-8_3.9x4.9mm_P1.27mm
Changed lines of the file:
@@
 F 0 "U5" H 5550 3750 50  0000 L CNN
 F 1 "PCA82C251" H 5550 3650 50  0000 L CNN
-F 2 "Housings_SOIC:SOIC-8_3.9x4.9mm_Pitch1.27mm" H 5750 3150 50  0001 C CNN
+F 2 "Package_SO:SO-8_3.9x4.9mm_P1.27mm" H 5750 3150 50  0001 C CNN
 F 3 "" H 5750 3150 50  0000 C CNN
 	1    5750 3200
@@
 F 0 "C9" H 6325 3850 50  0000 L CNN
 F 1 "100n" H 6325 3650 50  0000 L CNN
-F 2 "Capacitors_SMD:C_0805" H 6338 3600 50  0001 C CNN
+F 2 "Capacitor_SMD:C_0805_2012Metric" H 6338 3600 50  0001 C CNN
 F 3 "" H 6300 3750 50  0000 C CNN
 	1    6300 3750

Commit message: - changed ref divider to 1k
Parts:
- U5: symbol philips:PCA82C251 -> Revolter-rescue:PCA82C251-philips
Changed lines of the file:
@@
 CAN_RX
 $Comp
-L philips:PCA82C251 U5
+L Revolter-rescue:PCA82C251-philips U5
 U 1 1 59A31FD5
 P 5750 3200
