File: Power.sch (KiCad schematic (older format))
At the start: 38 parts, among them IC3 INA181A1, IC4 INA181A1, IC5 INA181A1, U2 IRS2186, U3 IRS2186, U4 IRS2186

Commit message: - changed ref divider to 1k
Parts:
- R45, R46: value 10k -> 1k
- U2, U3, U4: symbol Driver_FET:IRS2186 -> Revolter-rescue:IRS2186-Driver_FET
Changed lines of the file:
@@
 P 5600 1450
 F 0 "R45" V 5680 1450 50  0000 C CNN
-F 1 "10k" V 5600 1450 50  0000 C CNN
+F 1 "1k" V 5600 1450 50  0000 C CNN
 F 2 "Resistor_SMD:R_0805_2012Metric" V 5530 1450 50  0001 C CNN
 F 3 "" H 5600 1450 50  0000 C CNN
@@
 P 5600 2050
 F 0 "R46" V 5680 2050 50  0000 C CNN
-F 1 "10k" V 5600 2050 50  0000 C CNN
+F 1 "1k" V 5600 2050 50  0000 C CNN
 F 2 "Resistor_SMD:R_0805_2012Metric" V 5530 2050 50  0001 C CNN
 F 3 "" H 5600 2050 50  0000 C CNN
@@
 	5400 3650 5550 3650
 $Comp
-L Driver_FET:IRS2186 U2
+L Revolter-rescue:IRS2186-Driver_FET U2
 U 1 1 5C96735E
 P 1350 1550
+AR Path="/5C96735E" Ref="U2"  Part="1"
+AR Path="/5895E6A0/5C96735E" Ref="U2"  Part="1"
 F 0 "U2" H 1100 1200 50  0000 C CNN
 F 1 "IRS2186" H 1550 1200 50  0000 C CNN
@@
 	1800 2700 1650 2700
 $Comp
-L Driver_FET:IRS2186 U3
+L Revolter-rescue:IRS2186-Driver_FET U3
 U 1 1 5C99754B
 P 1350 2900
+AR Path="/5C99754B" Ref="U3"  Part="1"
+AR Path="/5895E6A0/5C99754B" Ref="U3"  Part="1"
 F 0 "U3" H 1100 2550 50  0000 C CNN
 F 1 "IRS2186" H 1550 2550 50  0000 C CNN
@@
 	1800 4050 1650 4050
 $Comp
-L Driver_FET:IRS2186 U4
+L Revolter-rescue:IRS2186-Driver_FET U4
 U 1 1 5C99AA3B
 P 1350 4250
+AR Path="/5C99AA3B" Ref="U4"  Part="1"
+AR Path="/5895E6A0/5C99AA3B" Ref="U4"  Part="1"
 F 0 "U4" H 1100 3900 50  0000 C CNN
 F 1 "IRS2186" H 1550 3900 50  0000 C CNN
