File: Power.sch (KiCad schematic (older format))
At the start: 49 parts, among them IC3 IRSM005, IC4 IRSM005, IC5 IRSM005, U2 ACS730xLCTR-50AB, U3 ACS730xLCTR-50AB, U4 ACS730xLCTR-50AB

Commit message: - added flyback diodes to FAN outputs - added fourth DC cap - changed TEMP3 to motor temp
Parts:
- added C7: CP, Capacitor_THT:CP_Radial_D6.3mm_P2.50mm, symbol Device:C_Polarized
- U2, U3, U4: value ACS730xLCTR-50AB -> ACS722LLCTR-40AU-T
Other:
- moved on the sheet: C26, C27, C29, C33, C34, C35, C36, C37, C38, C39, C40, C41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

Commit message: - updated current sensor value
Parts:
- U2, U3, U4: value ACS722LLCTR-40AU-T -> ACS722LLCTR-40AB-T
Changed lines of the file:
@@
 P 7550 3800
 F 0 "U4" V 7250 4150 50  0000 L CNN
-F 1 "ACS722LLCTR-40AU-T" V 7450 4100 50  0000 L CNN
+F 1 "ACS722LLCTR-40AB-T" V 7450 4100 50  0000 L CNN
 F 2 "Package_SO:SOIC-8_3.9x4.9mm_P1.27mm" H 7900 3700 50  0001 L CIN
 F 3 "http://www.allegromicro.com/~/media/Files/Datasheets/ACS730-Datasheet.ashx?la=en" H 7550 3800 50  0001 C CNN
@@
 P 3700 1550
 F 0 "U2" V 3400 1900 50  0000 L CNN
-F 1 "ACS722LLCTR-40AU-T" V 3600 1850 50  0000 L CNN
+F 1 "ACS722LLCTR-40AB-T" V 3600 1850 50  0000 L CNN
 F 2 "Package_SO:SOIC-8_3.9x4.9mm_P1.27mm" H 4050 1450 50  0001 L CIN
 F 3 "http://www.allegromicro.com/~/media/Files/Datasheets/ACS730-Datasheet.ashx?la=en" H 3700 1550 50  0001 C CNN
@@
 P 3700 6200
 F 0 "U3" V 3400 6550 50  0000 L CNN
-F 1 "ACS722LLCTR-40AU-T" V 3600 6500 50  0000 L CNN
+F 1 "ACS722LLCTR-40AB-T" V 3600 6500 50  0000 L CNN
 F 2 "Package_SO:SOIC-8_3.9x4.9mm_P1.27mm" H 4050 6100 50  0001 L CIN
 F 3 "http://www.allegromicro.com/~/media/Files/Datasheets/ACS730-Datasheet.ashx?la=en" H 3700 6200 50  0001 C CNN

Commit message: - removed one fan output - moved PWM pins to TIM4 - added pull-up to fan output (for 4pin fan) - removed blue power LED - split 12pin to 5 2pin connectors - reduced LED resistors - removed optional current sensor - removed HV DCDC converter - added some cap values
Parts:
- removed C15: 1u, Capacitor_SMD:C_0805_2012Metric, symbol Device:C
- removed JP2: 2SHUNT, Jumper:SolderJumper-2_P1.3mm_Open_TrianglePad1.0x1.5mm, symbol Jumper:SolderJumper_2_Open
- removed U4: ACS722LLCTR-40AB-T, Package_SO:SOIC-8_3.9x4.9mm_P1.27mm, symbol Sensor_Current:ACS722xLCTR-40AB
- C16, C17, C22, C7: value CP -> 100u/35V
- C26, C27, C29, C33, C34, C35, C36, C37, C38, C39, C40, C41, C42, C44, C50: value C -> 10u/50V
Connections:
- net labels removed: CURRENT_V
Changed lines of the file:
@@
 	1    0    0    -1
-$EndComp
-$Comp
-L Device:C C15
-U 1 1 5EF63647
-P 7950 3650
-F 0 "C15" H 7835 3604 50  0000 R CNN
-F 1 "1u" H 7835 3695 50  0000 R CNN
-F 2 "Capacitor_SMD:C_0805_2012Metric" H 7988 3500 50  0001 C CNN
-F 3 "~" H 7950 3650 50  0001 C CNN
-	1    7950 3650
-	-1   0    0    1
-$EndComp
-$Comp
-L power:GND #PWR0171
-U 1 1 5EF6364D
-P 7150 3800
-F 0 "#PWR0171" H 7150 3550 50  0001 C CNN
-F 1 "GND" V 7155 3672 50  0000 R CNN
-F 2 "" H 7150 3800 50  0001 C CNN
-F 3 "" H 7150 3800 50  0001 C CNN
-	1    7150 3800
-	0    1    1    0
-$EndComp
-$Comp
-L power:GND #PWR0172
-U 1 1 5EF63653
-P 7950 3500
-F 0 "#PWR0172" H 7950 3250 50  0001 C CNN
-F 1 "GND" H 7955 3327 50  0000 C CNN
-F 2 "" H 7950 3500 50  0001 C CNN
-F 3 "" H 7950 3500 50  0001 C CNN
-	1    7950 3500
-	-1   0    0    1
-$EndComp
-$Comp
-L power:+3V3 #PWR0173
-U 1 1 5EF63659
-P 7950 3800
-F 0 "#PWR0173" H 7950 3650 50  0001 C CNN
-F 1 "+3V3" V 7965 3928 50  0000 L CNN
-F 2 "" H 7950 3800 50  0001 C CNN
-F 3 "" H 7950 3800 50  0001 C CNN
-	1    7950 3800
-	0    1    1    0
 $EndComp
 Wire Wire Line
@@
 Wire Wire Line
 	8300 4200 7750 4200
-$Comp
-L power:GND #PWR0176
-U 1 1 5EF6367F
-P 7450 3400
-F 0 "#PWR0176" H 7450 3150 50  0001 C CNN
-F 1 "GND" H 7455 3227 50  0000 C CNN
-F 2 "" H 7450 3400 50  0001 C CNN
-F 3 "" H 7450 3400 50  0001 C CNN
-	1    7450 3400
-	-1   0    0    1
-$EndComp
-Text HLabel 7750 3400 1    60   Output ~ 0
-CURRENT_V
-$Comp
-L Sensor_Current:ACS722xLCTR-40AB U4
-U 1 1 5EEBCE46
-P 7550 3800
-F 0 "U4" V 7250 4150 50  0000 L CNN
-F 1 "ACS722LLCTR-40AB-T" V 7450 4100 50  0000 L CNN
-F 2 "Package_SO:SOIC-8_3.9x4.9mm_P1.27mm" H 7900 3700 50  0001 L CIN
-F 3 "http://www.allegromicro.com/~/media/Files/Datasheets/ACS730-Datasheet.ashx?la=en" H 7550 3800 50  0001 C CNN
-	1    7550 3800
-	0    1    -1   0
-$EndComp
 $Comp
 L Sensor_Current:ACS722xLCTR-40AB U2
@@
 U 1 1 5EF55DAC
 P 10400 1300
-F 0 "C16" H 10518 1346 50  0000 L CNN
-F 1 "CP" H 10518 1255 50  0000 L CNN
+F 0 "C16" V 10500 1450 50  0000 L CNN
+F 1 "100u/35V" V 10300 1450 50  0000 L CNN
 F 2 "Capacitor_THT:CP_Radial_D6.3mm_P2.50mm" H 10438 1150 50  0001 C CNN
 F 3 "~" H 10400 1300 50  0001 C CNN
@@
 U 1 1 5EF56825
 P 10750 1300
-F 0 "C17" H 10868 1346 50  0000 L CNN
-F 1 "CP" H 10868 1255 50  0000 L CNN
+F 0 "C17" V 10850 1450 50  0000 L CNN
+F 1 "100u/35V" V 10650 1450 50  0000 L CNN
 F 2 "Capacitor_THT:CP_Radial_D6.3mm_P2.50mm" H 10788 1150 50  0001 C CNN
 F 3 "~" H 10750 1300 50  0001 C CNN
@@
 U 1 1 5EF6711E
 P 10050 1300
-F 0 "C22" H 10168 1346 50  0000 L CNN
-F 1 "CP" H 10168 1255 50  0000 L CNN
+F 0 "C22" V 10150 1450 50  0000 L CNN
+F 1 "100u/35V" V 9950 1450 50  0000 L CNN
 F 2 "Capacitor_THT:CP_Radial_D6.3mm_P2.50mm" H 10088 1150 50  0001 C CNN
 F 3 "~" H 10050 1300 50  0001 C CNN
@@
 P 9200 1300
 F 0 "C40" V 9150 1350 50  0000 L CNN
-F 1 "C" V 9250 1350 50  0000 L CNN
+F 1 "10u/50V" V 9250 1350 50  0000 L CNN
 F 2 "Capacitor_SMD:C_1206_3216Metric" H 9238 1150 50  0001 C CNN
 F 3 "~" H 9200 1300 50  0001 C CNN
@@
 P 9000 1300
 F 0 "C39" V 8950 1350 50  0000 L CNN
-F 1 "C" V 9050 1350 50  0000 L CNN
+F 1 "10u/50V" V 9050 1350 50  0000 L CNN
 F 2 "Capacitor_SMD:C_1206_3216Metric" H 9038 1150 50  0001 C CNN
 F 3 "~" H 9000 1300 50  0001 C CNN
@@
 P 8800 1300
 F 0 "C38" V 8750 1350 50  0000 L CNN
-F 1 "C" V 8850 1350 50  0000 L CNN
+F 1 "10u/50V" V 8850 1350 50  0000 L CNN
 F 2 "Capacitor_SMD:C_1206_3216Metric" H 8838 1150 50  0001 C CNN
 F 3 "~" H 8800 1300 50  0001 C CNN
@@
 P 8600 1300
 F 0 "C37" V 8550 1350 50  0000 L CNN
-F 1 "C" V 8650 1350 50  0000 L CNN
+F 1 "10u/50V" V 8650 1350 50  0000 L CNN
 F 2 "Capacitor_SMD:C_1206_3216Metric" H 8638 1150 50  0001 C CNN
 F 3 "~" H 8600 1300 50  0001 C CNN
@@
 P 8400 1300
 F 0 "C36" V 8350 1350 50  0000 L CNN
-F 1 "C" V 8450 1350 50  0000 L CNN
+F 1 "10u/50V" V 8450 1350 50  0000 L CNN
 F 2 "Capacitor_SMD:C_1206_3216Metric" H 8438 1150 50  0001 C CNN
 F 3 "~" H 8400 1300 50  0001 C CNN
@@
 P 8200 1300
 F 0 "C35" V 8150 1350 50  0000 L CNN
-F 1 "C" V 8250 1350 50  0000 L CNN
+F 1 "10u/50V" V 8250 1350 50  0000 L CNN
 F 2 "Capacitor_SMD:C_1206_3216Metric" H 8238 1150 50  0001 C CNN
 F 3 "~" H 8200 1300 50  0001 C CNN
@@
 P 8000 1300
 F 0 "C34" V 7950 1350 50  0000 L CNN
-F 1 "C" V 8050 1350 50  0000 L CNN
+F 1 "10u/50V" V 8050 1350 50  0000 L CNN
 F 2 "Capacitor_SMD:C_1206_3216Metric" H 8038 1150 50  0001 C CNN
 F 3 "~" H 8000 1300 50  0001 C CNN
@@
 P 7800 1300
 F 0 "C33" V 7750 1350 50  0000 L CNN
-F 1 "C" V 7850 1350 50  0000 L CNN
+F 1 "10u/50V" V 7850 1350 50  0000 L CNN
 F 2 "Capacitor_SMD:C_1206_3216Metric" H 7838 1150 50  0001 C CNN
 F 3 "~" H 7800 1300 50  0001 C CNN
@@
 P 7600 1300
 F 0 "C29" V 7550 1350 50  0000 L CNN
-F 1 "C" V 7650 1350 50  0000 L CNN
+F 1 "10u/50V" V 7650 1350 50  0000 L CNN
 F 2 "Capacitor_SMD:C_1206_3216Metric" H 7638 1150 50  0001 C CNN
 F 3 "~" H 7600 1300 50  0001 C CNN
@@
 P 7400 1300
 F 0 "C27" V 7350 1350 50  0000 L CNN
-F 1 "C" V 7450 1350 50  0000 L CNN
+F 1 "10u/50V" V 7450 1350 50  0000 L CNN
 F 2 "Capacitor_SMD:C_1206_3216Metric" H 7438 1150 50  0001 C CNN
 F 3 "~" H 7400 1300 50  0001 C CNN
@@
 P 7200 1300
 F 0 "C26" V 7150 1350 50  0000 L CNN
-F 1 "C" V 7250 1350 50  0000 L CNN
+F 1 "10u/50V" V 7250 1350 50  0000 L CNN
 F 2 "Capacitor_SMD:C_1206_3216Metric" H 7238 1150 50  0001 C CNN
 F 3 "~" H 7200 1300 50  0001 C CNN
@@
 P 7000 1300
 F 0 "C50" V 6950 1350 50  0000 L CNN
-F 1 "C" V 7050 1350 50  0000 L CNN
+F 1 "10u/50V" V 7050 1350 50  0000 L CNN
 F 2 "Capacitor_SMD:C_1206_3216Metric" H 7038 1150 50  0001 C CNN
 F 3 "~" H 7000 1300 50  0001 C CNN
@@
 P 6800 1300
 F 0 "C44" V 6750 1350 50  0000 L CNN
-F 1 "C" V 6850 1350 50  0000 L CNN
+F 1 "10u/50V" V 6850 1350 50  0000 L CNN
 F 2 "Capacitor_SMD:C_1206_3216Metric" H 6838 1150 50  0001 C CNN
 F 3 "~" H 6800 1300 50  0001 C CNN
@@
 P 6600 1300
 F 0 "C42" V 6550 1350 50  0000 L CNN
-F 1 "C" V 6650 1350 50  0000 L CNN
+F 1 "10u/50V" V 6650 1350 50  0000 L CNN
 F 2 "Capacitor_SMD:C_1206_3216Metric" H 6638 1150 50  0001 C CNN
 F 3 "~" H 6600 1300 50  0001 C CNN
@@
 P 6400 1300
 F 0 "C41" V 6350 1350 50  0000 L CNN
-F 1 "C" V 6450 1350 50  0000 L CNN
+F 1 "10u/50V" V 6450 1350 50  0000 L CNN
 F 2 "Capacitor_SMD:C_1206_3216Metric" H 6438 1150 50  0001 C CNN
 F 3 "~" H 6400 1300 50  0001 C CNN
@@
 $EndComp
 $Comp
-L Jumper:SolderJumper_2_Open JP2
-U 1 1 5F5CEC3F
-P 7600 4200
-F 0 "JP2" H 7600 4385 50  0000 C CNN
-F 1 "2SHUNT" H 7550 4100 50  0000 C CNN
-F 2 "Jumper:SolderJumper-2_P1.3mm_Open_TrianglePad1.0x1.5mm" H 7600 4200 50  0001 C CNN
-F 3 "~" H 7600 4200 50  0001 C CNN
-	1    7600 4200
-	1    0    0    -1
-$EndComp
-$Comp
 L Sensor_Current:ACS722xLCTR-40AB U3
 U 1 1 5EEC028C
@@
 	0    1    -1   0
 $EndComp
-Connection ~ 7750 4200
 Wire Wire Line
 	7750 4200 7750 4450
-Wire Wire Line
-	6350 4200 7450 4200
-Connection ~ 7450 4200
-Connection ~ 7950 3800
 Connection ~ 4100 1550
 Connection ~ 3900 1950
@@
 U 1 1 5FCB7911
 P 9700 1300
-F 0 "C7" H 9818 1346 50  0000 L CNN
-F 1 "CP" H 9818 1255 50  0000 L CNN
+F 0 "C7" V 9800 1450 50  0000 L CNN
+F 1 "100u/35V" V 9600 1450 50  0000 L CNN
 F 2 "Capacitor_THT:CP_Radial_D6.3mm_P2.50mm" H 9738 1150 50  0001 C CNN
 F 3 "~" H 9700 1300 50  0001 C CNN
@@
 	1    0    0    -1
 $EndComp
+Connection ~ 5050 4150
+Connection ~ 1200 1900
+Wire Wire Line
+	6350 4200 7750 4200
+Connection ~ 7750 4200
 $EndSCHEMATC
