File: Revolter.sch (KiCad schematic (older format))
At the start: 24 parts, among them P1 USB_B, P2 Interface, P3 IN+, P4 IN-, P5 MOTOR3, P6 MOTOR2, P7 MOTOR1

Commit message: - removed 1 MOSFET of each group (no space) - removed 2 DC buffer caps (no space) - power stage routed - shunts and amps routed - post driver routed - pre driver HV routed
Parts:
- removed C1: 100n, Capacitors_SMD:C_0805, symbol C-RESCUE-BLDC_4
- removed D1: SS14, Diodes_SMD:SMA_Standard, symbol D_Schottky_Small
- removed P2: Interface, alexmod:XG4A_20_wo_56, symbol CONN_01X18_20
- removed R3: 2k2, Resistors_SMD:R_0805, symbol R-RESCUE-BLDC_4
- added D13: 3V3, Diodes_SMD:D_SOD-123, symbol ZENER
- added P10: AUX, Connectors_Terminal_Blocks:TerminalBlock_Pheonix_PT-3.5mm_7pol, symbol CONN_01X07
- added P2: CAN, Connectors_Terminal_Blocks:TerminalBlock_Pheonix_PT-3.5mm_4pol, symbol CONN_01X04
- added P9: Motor, Connectors_Terminal_Blocks:TerminalBlock_Pheonix_PT-3.5mm_6pol, symbol CONN_01X06
- P1: footprint alexmod:USBB_vert -> Connectors_USB:USB_Micro-B_Molex-105017-0001
- P3, P4, P5, P6, P7: footprint Mounting_Holes:MountingHole_6.5mm_Pad_Via -> Mounting_Holes:MountingHole_3.2mm_M3_Pad_Via
- R7: value 160k -> 100k
Connections:
- net labels removed: Earth
- wire segments 79 -> 81
- no-connect marks 1 -> 0
Other:
- note removed: "100R if used as\nservo output"

Commit message: - redesigned the MOSFET mounting -> minor changes to the power stage - logic and interface routed -> layout finished - needs final check and gerber export
Parts:
- removed R11: R, Resistors_SMD:R_0805, symbol R
- added JP1: JUMPER, alexmod:Jumper_2, symbol JUMPER
Connections:
- net labels added: +12V
- net labels removed: +12VA
Changed lines of the file:
@@
 L GND-RESCUE-BLDC_4 #PWR01
 U 1 1 5895E67B
-P 8850 4900
-F 0 "#PWR01" H 8850 4900 30  0001 C CNN
-F 1 "GND" H 8850 4830 30  0001 C CNN
-F 2 "" H 8850 4900 60  0001 C CNN
-F 3 "" H 8850 4900 60  0001 C CNN
-	1    8850 4900
+P 8550 4900
+F 0 "#PWR01" H 8550 4900 30  0001 C CNN
+F 1 "GND" H 8550 4830 30  0001 C CNN
+F 2 "" H 8550 4900 60  0001 C CNN
+F 3 "" H 8550 4900 60  0001 C CNN
+	1    8550 4900
 	1    0    0    -1
 $EndComp
@@
 C8 C8 08 D2 A9 87 39 1B F9 3D 64 10 3C A5 22 3B 19 76 2F 98 2B 2B 2B 1E 8F A7 AB AB 0B FB AC 1D
 B9 73 C8 EF 2C EC 8D 33 57 03 96 70 05 29 43 0C 6A C5 A8 D7 30 9E 87 2D DE BE E8 EA 73 2F 9C 18
-F1 B3 C3 9F 6D FA 1E FF 03 71 17 46 7E 55 DF FF 4E 00 00 00 00 49 45 4E 44 AE 42 60 82 2B
+F1 B3 C3 9F 6D FA 1E FF 03 71 17 46 7E 55 DF FF 4E 00 00 00 00 49 45 4E 44 AE 42 60 82 F8
 EndData
 $EndBitmap
@@
 	7650 3900 8300 3900
 Wire Wire Line
-	8850 4800 8850 4900
+	8550 4800 8550 4900
 Wire Wire Line
 	9150 4800 9150 4900
@@
 $EndComp
 $Comp
-L R R11
-U 1 1 5895E6AC
-P 9000 4800
-F 0 "R11" V 9080 4800 50  0000 C CNN
-F 1 "R" V 9000 4800 50  0000 C CNN
-F 2 "Resistors_SMD:R_0805" V 8930 4800 30  0001 C CNN
-F 3 "" H 9000 4800 30  0000 C CNN
-	1    9000 4800
-	0    1    1    0
-$EndComp
-$Comp
 L GNDPWR #PWR06
 U 1 1 5895E6AD
@@
 20 08 82 84 0E 7A 08 41 10 04 29 27 E8 21 04 41 10 A4 9C A0 87 10 04 41 90 72 82 1E 42 10 04 41
 CA 09 7A 08 41 10 04 29 27 E8 21 04 41 10 A4 9C FC 1F 60 28 4A EE 61 E4 B4 21 00 00 00 00 49 45
-4E 44 AE 42 60 82 7F
+4E 44 AE 42 60 82 9C
 EndData
 $EndBitmap
@@
 	0    1    1    0
 $EndComp
-$Comp
-L +12VA #PWR015
-U 1 1 5899E265
-P 1350 3650
-F 0 "#PWR015" H 1350 3500 50  0001 C CNN
-F 1 "+12VA" H 1350 3790 50  0000 C CNN
-F 2 "" H 1350 3650 60  0000 C CNN
-F 3 "" H 1350 3650 60  0000 C CNN
-	1    1350 3650
-	1    0    0    -1
-$EndComp
 Wire Wire Line
 	1350 3650 1350 3700
@@
 Wire Wire Line
 	1450 5000 1300 5000
+$Comp
+L JUMPER JP1
+U 1 1 59C3E8D3
+P 8850 4800
+F 0 "JP1" H 8850 4950 50  0000 C CNN
+F 1 "JUMPER" H 8850 4720 50  0000 C CNN
+F 2 "alexmod:Jumper_2" H 8850 4800 50  0001 C CNN
+F 3 "" H 8850 4800 50  0000 C CNN
+	1    8850 4800
+	1    0    0    -1
+$EndComp
+$Comp
+L +12V #PWR?
+U 1 1 59C48CD0
+P 1350 3650
+F 0 "#PWR?" H 1350 3500 50  0001 C CNN
+F 1 "+12V" H 1350 3790 50  0000 C CNN
+F 2 "" H 1350 3650 50  0000 C CNN
+F 3 "" H 1350 3650 50  0000 C CNN
+	1    1350 3650
+	1    0    0    -1
+$EndComp
 $EndSCHEMATC

Commit message: - final check - minor layout cleanups - labeling - first production run => V1.0
Parts:
- removed P1: USB_B, Connectors_USB:USB_Micro-B_Molex-105017-0001, symbol USB_B
- added P1: USB_OTG, Connectors_USB:USB_Micro-B_Molex-105017-0001, symbol USB_OTG
Changed lines of the file:
@@
 C8 C8 08 D2 A9 87 39 1B F9 3D 64 10 3C A5 22 3B 19 76 2F 98 2B 2B 2B 1E 8F A7 AB AB 0B FB AC 1D
 B9 73 C8 EF 2C EC 8D 33 57 03 96 70 05 29 43 0C 6A C5 A8 D7 30 9E 87 2D DE BE E8 EA 73 2F 9C 18
-F1 B3 C3 9F 6D FA 1E FF 03 71 17 46 7E 55 DF FF 4E 00 00 00 00 49 45 4E 44 AE 42 60 82 F8
+F1 B3 C3 9F 6D FA 1E FF 03 71 17 46 7E 55 DF FF 4E 00 00 00 00 49 45 4E 44 AE 42 60 82 3E
 EndData
 $EndBitmap
@@
 20 08 82 84 0E 7A 08 41 10 04 29 27 E8 21 04 41 10 A4 9C A0 87 10 04 41 90 72 82 1E 42 10 04 41
 CA 09 7A 08 41 10 04 29 27 E8 21 04 41 10 A4 9C FC 1F 60 28 4A EE 61 E4 B4 21 00 00 00 00 49 45
-4E 44 AE 42 60 82 9C
+4E 44 AE 42 60 82 7C
 EndData
 $EndBitmap
@@
 $EndComp
 $Comp
-L USB_B P1
-U 1 1 5899E24E
-P 950 3050
-F 0 "P1" H 1150 2850 50  0000 C CNN
-F 1 "USB_B" H 900 3250 50  0000 C CNN
-F 2 "Connectors_USB:USB_Micro-B_Molex-105017-0001" V 900 2950 60  0001 C CNN
-F 3 "" V 900 2950 60  0000 C CNN
-	1    950  3050
-	0    -1   1    0
-$EndComp
-$Comp
 L GND-RESCUE-BLDC_4 #PWR013
 U 1 1 5899E24F
-P 1250 3150
-F 0 "#PWR013" H 1250 3150 30  0001 C CNN
-F 1 "GND" H 1250 3080 30  0001 C CNN
-F 2 "" H 1250 3150 60  0001 C CNN
-F 3 "" H 1250 3150 60  0001 C CNN
-	1    1250 3150
+P 1250 3250
+F 0 "#PWR013" H 1250 3250 30  0001 C CNN
+F 1 "GND" H 1250 3180 30  0001 C CNN
+F 2 "" H 1250 3250 60  0001 C CNN
+F 3 "" H 1250 3250 60  0001 C CNN
+	1    1250 3250
 	0    -1   1    0
 $EndComp
@@
 L GND-RESCUE-BLDC_4 #PWR014
 U 1 1 5899E250
-P 850 3350
-F 0 "#PWR014" H 850 3350 30  0001 C CNN
-F 1 "GND" H 850 3280 30  0001 C CNN
-F 2 "" H 850 3350 60  0001 C CNN
-F 3 "" H 850 3350 60  0001 C CNN
-	1    850  3350
+P 850 3450
+F 0 "#PWR014" H 850 3450 30  0001 C CNN
+F 1 "GND" H 850 3380 30  0001 C CNN
+F 2 "" H 850 3450 60  0001 C CNN
+F 3 "" H 850 3450 60  0001 C CNN
+	1    850  3450
 	-1   0    0    -1
 $EndComp
@@
 	5200 4500 5200 4550
 $Comp
-L GND-RESCUE-BLDC_4 #PWR016
+L GND-RESCUE-BLDC_4 #PWR015
 U 1 1 599AD91E
 P 5450 4900
-F 0 "#PWR016" H 5450 4900 30  0001 C CNN
+F 0 "#PWR015" H 5450 4900 30  0001 C CNN
 F 1 "GND" H 5450 4830 30  0001 C CNN
 F 2 "" H 5450 4900 60  0001 C CNN
@@
 $EndComp
 $Comp
-L GND-RESCUE-BLDC_4 #PWR017
+L GND-RESCUE-BLDC_4 #PWR016
 U 1 1 59A3EB3E
 P 1300 4000
-F 0 "#PWR017" H 1300 4000 30  0001 C CNN
+F 0 "#PWR016" H 1300 4000 30  0001 C CNN
 F 1 "GND" H 1300 3930 30  0001 C CNN
 F 2 "" H 1300 4000 60  0001 C CNN
@@
 $EndComp
 $Comp
-L GND-RESCUE-BLDC_4 #PWR018
+L GND-RESCUE-BLDC_4 #PWR017
 U 1 1 59A41697
 P 1300 4800
-F 0 "#PWR018" H 1300 4800 30  0001 C CNN
+F 0 "#PWR017" H 1300 4800 30  0001 C CNN
 F 1 "GND" H 1300 4730 30  0001 C CNN
 F 2 "" H 1300 4800 60  0001 C CNN
@@
 $EndComp
 $Comp
-L +5V #PWR019
+L +5V #PWR018
 U 1 1 59A4AB16
 P 1350 4250
-F 0 "#PWR019" H 1350 4100 50  0001 C CNN
+F 0 "#PWR018" H 1350 4100 50  0001 C CNN
 F 1 "+5V" H 1350 4390 50  0000 C CNN
 F 2 "" H 1350 4250 50  0000 C CNN
@@
 	2950 5500 1300 5500
 $Comp
-L GND-RESCUE-BLDC_4 #PWR020
+L GND-RESCUE-BLDC_4 #PWR019
 U 1 1 59A5655A
 P 1300 5600
-F 0 "#PWR020" H 1300 5600 30  0001 C CNN
+F 0 "#PWR019" H 1300 5600 30  0001 C CNN
 F 1 "GND" H 1300 5530 30  0001 C CNN
 F 2 "" H 1300 5600 60  0001 C CNN
@@
 $EndComp
 $Comp
-L +3V3 #PWR021
+L +3V3 #PWR020
 U 1 1 59A596B5
 P 1450 4950
-F 0 "#PWR021" H 1450 4800 50  0001 C CNN
+F 0 "#PWR020" H 1450 4800 50  0001 C CNN
 F 1 "+3V3" H 1450 5090 50  0000 C CNN
 F 2 "" H 1450 4950 60  0000 C CNN
@@
 $EndComp
 $Comp
-L +12V #PWR?
+L +12V #PWR021
 U 1 1 59C48CD0
 P 1350 3650
-F 0 "#PWR?" H 1350 3500 50  0001 C CNN
+F 0 "#PWR021" H 1350 3500 50  0001 C CNN
 F 1 "+12V" H 1350 3790 50  0000 C CNN
 F 2 "" H 1350 3650 50  0000 C CNN
@@
 	1    0    0    -1
 $EndComp
+$Comp
+L USB_OTG P1
+U 1 1 59C54C98
+P 950 3050
+F 0 "P1" H 1275 2925 50  0000 C CNN
+F 1 "USB_OTG" H 950 3250 50  0000 C CNN
+F 2 "Connectors_USB:USB_Micro-B_Molex-105017-0001" V 900 2950 50  0001 C CNN
+F 3 "" V 900 2950 50  0000 C CNN
+	1    950  3050
+	0    -1   1    0
+$EndComp
 $EndSCHEMATC

Commit message: - fixed swapped pins 2 and 3 on IC2 - added optional dividers to ADC inputs - made Vcc selectable between 3V3 or 5V
Parts:
- added JP2: Vcc select, Pin_Headers:Pin_Header_Straight_1x03_Pitch2.54mm, symbol Jumper_NC_Dual
- added JP3, JP4: opt., alexmod:Jumper_2, symbol Jumper_NC_Small
- added R11, R61: 1k, Resistors_SMD:R_0805, symbol R
- added R62, R63: 1k5, Resistors_SMD:R_0805, symbol R
- D13: symbol ZENER -> ZENER-RESCUE-Revolter
- P1: symbol USB_OTG -> USB_OTG-RESCUE-Revolter
Connections:
- wire segments 81 -> 91
Changed lines of the file:
@@
 C8 C8 08 D2 A9 87 39 1B F9 3D 64 10 3C A5 22 3B 19 76 2F 98 2B 2B 2B 1E 8F A7 AB AB 0B FB AC 1D
 B9 73 C8 EF 2C EC 8D 33 57 03 96 70 05 29 43 0C 6A C5 A8 D7 30 9E 87 2D DE BE E8 EA 73 2F 9C 18
-F1 B3 C3 9F 6D FA 1E FF 03 71 17 46 7E 55 DF FF 4E 00 00 00 00 49 45 4E 44 AE 42 60 82 3E
+F1 B3 C3 9F 6D FA 1E FF 03 71 17 46 7E 55 DF FF 4E 00 00 00 00 49 45 4E 44 AE 42 60 82
 EndData
 $EndBitmap
@@
 20 08 82 20 08 12 3C 28 79 08 82 20 08 82 20 2D 08 4A 1E 82 20 08 82 20 48 0B 82 92 87 20 08 82
 20 08 D2 82 A0 E4 21 08 82 20 08 82 B4 20 28 79 08 82 20 08 82 20 2D 08 4A 1E 82 20 08 82 20 48
-0B F2 FF 19 12 7F 86 40 CA 02 9D 00 00 00 00 49 45 4E 44 AE 42 60 82 00
+0B F2 FF 19 12 7F 86 40 CA 02 9D 00 00 00 00 49 45 4E 44 AE 42 60 82
 EndData
 $EndBitmap
@@
 20 08 82 84 0E 7A 08 41 10 04 29 27 E8 21 04 41 10 A4 9C A0 87 10 04 41 90 72 82 1E 42 10 04 41
 CA 09 7A 08 41 10 04 29 27 E8 21 04 41 10 A4 9C FC 1F 60 28 4A EE 61 E4 B4 21 00 00 00 00 49 45
-4E 44 AE 42 60 82 7C
+4E 44 AE 42 60 82
 EndData
 $EndBitmap
@@
 	5950 3600 5950 6300
 $Comp
-L ZENER D13
+L ZENER-RESCUE-Revolter D13
 U 1 1 599A9D56
 P 5450 4700
@@
 $EndComp
 Wire Wire Line
-	2950 5100 1300 5100
-Wire Wire Line
 	1300 5200 2950 5200
 Wire Wire Line
 	2950 5300 1300 5300
 Wire Wire Line
-	1300 5400 2950 5400
-Wire Wire Line
 	2950 5500 1300 5500
 $Comp
@@
 L +3V3 #PWR020
 U 1 1 59A596B5
-P 1450 4950
-F 0 "#PWR020" H 1450 4800 50  0001 C CNN
-F 1 "+3V3" H 1450 5090 50  0000 C CNN
-F 2 "" H 1450 4950 60  0000 C CNN
-F 3 "" H 1450 4950 60  0000 C CNN
-	1    1450 4950
-	1    0    0    -1
+P 1700 5950
+F 0 "#PWR020" H 1700 5800 50  0001 C CNN
+F 1 "+3V3" H 1700 6090 50  0000 C CNN
+F 2 "" H 1700 5950 60  0000 C CNN
+F 3 "" H 1700 5950 60  0000 C CNN
+	1    1700 5950
+	0    1    1    0
 $EndComp
 Wire Wire Line
-	1450 4950 1450 5000
-Wire Wire Line
 	1450 5000 1300 5000
 $Comp
@@
 $EndComp
 $Comp
-L USB_OTG P1
+L USB_OTG-RESCUE-Revolter P1
 U 1 1 59C54C98
 P 950 3050
@@
 	0    -1   1    0
 $EndComp
+$Comp
+L R R11
+U 1 1 5A8A2804
+P 1750 5100
+F 0 "R11" V 1830 5100 50  0000 C CNN
+F 1 "1k" V 1750 5100 50  0000 C CNN
+F 2 "Resistors_SMD:R_0805" V 1680 5100 50  0001 C CNN
+F 3 "" H 1750 5100 50  0001 C CNN
+	1    1750 5100
+	0    1    1    0
+$EndComp
+$Comp
+L R R61
+U 1 1 5A8A2AC4
+P 1750 5400
+F 0 "R61" V 1830 5400 50  0000 C CNN
+F 1 "1k" V 1750 5400 50  0000 C CNN
+F 2 "Resistors_SMD:R_0805" V 1680 5400 50  0001 C CNN
+F 3 "" H 1750 5400 50  0001 C CNN
+	1    1750 5400
+	0    1    1    0
+$EndComp
+$Comp
+L R R62
+U 1 1 5A8A2D56
+P 2050 5900
+F 0 "R62" V 2130 5900 50  0000 C CNN
+F 1 "1k5" V 2050 5900 50  0000 C CNN
+F 2 "Resistors_SMD:R_0805" V 1980 5900 50  0001 C CNN
+F 3 "" H 2050 5900 50  0001 C CNN
+	1    2050 5900
+	-1   0    0    1
+$EndComp
+$Comp
+L R R63
+U 1 1 5A8A304D
+P 2250 5900
+F 0 "R63" V 2330 5900 50  0000 C CNN
+F 1 "1k5" V 2250 5900 50  0000 C CNN
+F 2 "Resistors_SMD:R_0805" V 2180 5900 50  0001 C CNN
+F 3 "" H 2250 5900 50  0001 C CNN
+	1    2250 5900
+	-1   0    0    1
+$EndComp
+Wire Wire Line
+	1300 5100 1600 5100
+Wire Wire Line
+	1600 5400 1300 5400
+Wire Wire Line
+	1900 5400 2950 5400
+Wire Wire Line
+	1900 5100 2950 5100
+Wire Wire Line
+	2050 4950 2050 5750
+Connection ~ 2050 5100
+Wire Wire Line
+	2250 5400 2250 5750
+Connection ~ 2250 5400
+$Comp
+L GND-RESCUE-BLDC_4 #PWR022
+U 1 1 5A8A3C1F
+P 2050 6050
+F 0 "#PWR022" H 2050 6050 30  0001 C CNN
+F 1 "GND" H 2050 5980 30  0001 C CNN
+F 2 "" H 2050 6050 60  0001 C CNN
+F 3 "" H 2050 6050 60  0001 C CNN
+	1    2050 6050
+	-1   0    0    -1
+$EndComp
+$Comp
+L GND-RESCUE-BLDC_4 #PWR023
+U 1 1 5A8A3EAD
+P 2250 6050
+F 0 "#PWR023" H 2250 6050 30  0001 C CNN
+F 1 "GND" H 2250 5980 30  0001 C CNN
+F 2 "" H 2250 6050 60  0001 C CNN
+F 3 "" H 2250 6050 60  0001 C CNN
+	1    2250 6050
+	-1   0    0    -1
+$EndComp
+$Comp
+L Jumper_NC_Dual JP2
+U 1 1 5A8A998C
+P 1450 5950
+F 0 "JP2" H 1500 5850 50  0000 L CNN
+F 1 "Vcc select" H 1450 6050 50  0000 C BNN
+F 2 "Pin_Headers:Pin_Header_Straight_1x03_Pitch2.54mm" H 1450 5950 50  0001 C CNN
+F 3 "" H 1450 5950 50  0001 C CNN
+	1    1450 5950
+	-1   0    0    1
+$EndComp
+Wire Wire Line
+	1450 5850 1450 5000
+$Comp
+L +5V #PWR024
+U 1 1 5A8AF6D2
+P 1200 5950
+F 0 "#PWR024" H 1200 5800 50  0001 C CNN
+F 1 "+5V" H 1200 6090 50  0000 C CNN
+F 2 "" H 1200 5950 50  0000 C CNN
+F 3 "" H 1200 5950 50  0000 C CNN
+	1    1200 5950
+	0    -1   -1   0
+$EndComp
+$Comp
+L Jumper_NC_Small JP4
+U 1 1 5A8B7EC7
+P 1750 5650
+F 0 "JP4" H 1750 5730 50  0000 C CNN
+F 1 "opt." H 1760 5590 50  0000 C CNN
+F 2 "alexmod:Jumper_2" H 1750 5650 50  0001 C CNN
+F 3 "" H 1750 5650 50  0001 C CNN
+	1    1750 5650
+	1    0    0    -1
+$EndComp
+$Comp
+L Jumper_NC_Small JP3
+U 1 1 5A8B83EA
+P 1750 4950
+F 0 "JP3" H 1750 5030 50  0000 C CNN
+F 1 "opt." H 1760 4890 50  0000 C CNN
+F 2 "alexmod:Jumper_2" H 1750 4950 50  0001 C CNN
+F 3 "" H 1750 4950 50  0001 C CNN
+	1    1750 4950
+	1    0    0    -1
+$EndComp
+Wire Wire Line
+	1650 4950 1550 4950
+Wire Wire Line
+	1550 4950 1550 5100
+Connection ~ 1550 5100
+Wire Wire Line
+	1850 4950 2050 4950
+Wire Wire Line
+	1550 5400 1550 5650
+Wire Wire Line
+	1550 5650 1650 5650
+Connection ~ 1550 5400
+Wire Wire Line
+	1850 5650 2250 5650
+Connection ~ 2250 5650
 $EndSCHEMATC

Commit message: - basis commit for V1.1 - did an great overhaul of high current paths - fixed wrong 3V3 reg pin out - blew the IO connector up to 8 pins (turns out 7pin is rare) - changed shunt to 2512 - changed hf caps to double 1210 - two input caps - pin outs for all IO on silk screen - spread the references so you can actually read them - connected the Hall/Temp pull-ups to 3V3 instead of 5V - changed vias to 0.6/0.3mm - changed text to V1.1
Parts:
- removed JP2: Vcc select, Pin_Headers:Pin_Header_Straight_1x03_Pitch2.54mm, symbol Jumper_NC_Dual
- removed P10: AUX, Connectors_Terminal_Blocks:TerminalBlock_Pheonix_PT-3.5mm_7pol, symbol CONN_01X07
- added J1: IO, Connectors_Terminal_Blocks:TerminalBlock_Pheonix_PT-3.5mm_8pol, symbol Conn_01x08
- added JP2, JP5: opt., alexmod:Jumper_2, symbol Jumper_NC_Small

Commit message: - updated project to 5.0.0 - added some more ignores
Parts:
- C2: symbol C -> Device:C
- D13: symbol ZENER-RESCUE-Revolter -> Revolter-rescue:ZENER-RESCUE-Revolter
- D2, D3, D4: symbol LED-RESCUE-BLDC_4 -> Revolter-rescue:LED-RESCUE-BLDC_4
- J1: symbol Conn_01x08 -> conn:Conn_01x08
- JP1: symbol JUMPER -> Revolter-rescue:JUMPER
- JP2, JP3, JP4, JP5: symbol Jumper_NC_Small -> Device:Jumper_NC_Small
- P1: symbol USB_OTG-RESCUE-Revolter -> Revolter-rescue:USB_OTG-RESCUE-Revolter
- P2: symbol CONN_01X04 -> Revolter-rescue:CONN_01X04
- P3, P4, P5, P6, P7: symbol CONN_1 -> Revolter-rescue:CONN_1
- P9: symbol CONN_01X06 -> Revolter-rescue:CONN_01X06
- R1, R11, R2, R61, R62, R63, R7, R8: symbol R -> Device:R
- R10, R4, R5, R6, R9: symbol R-RESCUE-BLDC_4 -> Revolter-rescue:R-RESCUE-BLDC_4
Connections:
- wire segments 91 -> 96

Commit message: - swapped TO220 dual MOSFET for single DualCool88 MOSFET package - removed postdriver - changed IRS2110 for IRS2186 - added third shunt - rewired CPU for VESC6 compatibility - layout completely from scratch
Parts:
- removed JP1: JUMPER, alexmod:Jumper_2, symbol Revolter-rescue:JUMPER
- removed JP2, JP5: opt., alexmod:Jumper_2, symbol Device:Jumper_NC_Small
- removed P1: USB_OTG, Connectors_USB:USB_Micro-B_Molex-105017-0001, symbol Revolter-rescue:USB_OTG-RESCUE-Revolter
- added J2: USB_A, Connector_USB:USB_B_TE_5787834_Vertical, symbol conn:USB_A
- added JP1: Jumper_NC_Dual, Jumper:SolderJumper-3_P1.3mm_Open_RoundedPad1.0x1.5mm, symbol Device:Jumper_NC_Dual
- added NT1: Net-Tie_2, NetTie:NetTie-2_SMD_Pad0.5mm, symbol Device:Net-Tie_2
- C2: footprint Capacitors_SMD:C_0805 -> Capacitor_SMD:C_0805_2012Metric
- D13: footprint Diodes_SMD:D_SOD-123 -> Diode_SMD:D_SOD-123
- D2, D3, D4: footprint LEDs:LED_0805 -> LED_SMD:LED_0805_2012Metric
- J1: footprint Connectors_Terminal_Blocks:TerminalBlock_Pheonix_PT-3.5mm_8pol -> Connector_Phoenix_MC:PhoenixContact_MCV_1,5_8-G-3.5_1x08_P3.50mm_Vertical
- JP3, JP4: footprint alexmod:Jumper_2 -> Jumper:SolderJumper-2_P1.3mm_Open_RoundedPad1.0x1.5mm
- P2: footprint Connectors_Terminal_Blocks:TerminalBlock_Pheonix_PT-3.5mm_4pol -> Connector_Phoenix_MC:PhoenixContact_MCV_1,5_4-G-3.5_1x04_P3.50mm_Vertical
- P3, P4, P5, P6, P7: footprint Mounting_Holes:MountingHole_3.2mm_M3_Pad_Via -> MountingHole:MountingHole_3.2mm_M3_Pad_Via
- P9: footprint Connectors_Terminal_Blocks:TerminalBlock_Pheonix_PT-3.5mm_6pol -> Connector_Phoenix_MC:PhoenixContact_MCV_1,5_6-G-3.5_1x06_P3.50mm_Vertical
- R1, R10, R11, R2, R5, R6, R61, R62, R63, R7, R8: footprint Resistors_SMD:R_0805 -> Resistor_SMD:R_0805_2012Metric
- R4: value 2k2 -> 470R; footprint Resistors_SMD:R_0805 -> Resistor_SMD:R_0805_2012Metric
- R9: footprint Resistors_SMD:R_0603 -> Resistor_SMD:R_0603_1608Metric
Connections:
- wire segments 96 -> 90
Other:
- note added: "REVOLTER 100V"
- note removed: "Connect signal ground and\npower ground in one place only"
- note removed: "HSWR V2.0 100V"
- moved on the sheet: P7

Commit message: - changed ref divider to 1k
Parts:
- J1: symbol conn:Conn_01x08 -> Revolter-rescue:Conn_01x08-conn
- J2: symbol conn:USB_A -> Revolter-rescue:USB_A-conn
Changed lines of the file:
@@
 Connection ~ 2250 5750
 $Comp
-L conn:Conn_01x08 J1
+L Revolter-rescue:Conn_01x08-conn J1
 U 1 1 5AA57034
 P 1100 5400
@@
 	1450 5950 1450 5100
 $Comp
-L conn:USB_A J2
+L Revolter-rescue:USB_A-conn J2
 U 1 1 5C9CAE08
 P 950 2950
